Commit message: first step to ns in gz

File: urdf/bcr_bot.xacro (robot description, xacro)
@@ -210,5 +210,5 @@
         </inertial>
     </link>
-    <joint name="roof joint" type="fixed">
+    <joint name="roof_joint" type="fixed">
         <parent link="chassis_link"/>
         <child link="roof_link"/>

File: urdf/bcr_bot_ns.xacro (robot description, xacro)
@@ -210,5 +210,5 @@
         </inertial>
     </link>
-    <joint name="roof joint" type="fixed">
+    <joint name="roof_joint" type="fixed">
         <parent link="chassis_link"/>
         <child link="roof_link"/>

File: urdf/gz_ns.xacro (robot description, xacro)
@@ -20,8 +20,8 @@
             <odom_publish_frequency>30</odom_publish_frequency>
             <!-- Topics con namespace del robot -->
-            <topic>/model/$(arg robot_namespace)/cmd_vel</topic>
+            <topic>$(arg robot_namespace)/cmd_vel</topic>
             <xacro:if value="${odometry_source == 'encoders'}">
-                <odom_topic>/model/$(arg robot_namespace)/odometry</odom_topic>
-                <tf_topic>/model/$(arg robot_namespace)/tf</tf_topic>
+                <odom_topic>$(arg robot_namespace)/odometry</odom_topic>
+                <tf_topic>$(arg robot_namespace)/tf</tf_topic>
             </xacro:if>
             <!-- Frames con namespace -->
@@ -39,6 +39,6 @@
             <robot_base_frame>$(arg robot_namespace)/base_footprint</robot_base_frame>
             <!-- Topics con namespace -->
-            <odom_topic>/model/$(arg robot_namespace)/odometry</odom_topic>
-            <tf_topic>/model/$(arg robot_namespace)/tf</tf_topic>
+            <odom_topic>$(arg robot_namespace)/odometry</odom_topic>
+            <tf_topic>$(arg robot_namespace)/tf</tf_topic>
             <dimensions>2</dimensions>
             <odom_publish_frequency>10</odom_publish_frequency>
@@ -51,5 +51,5 @@
             <sensor name='gpu_lidar' type='gpu_lidar'>
                 <!-- Topic con namespace -->
-                <topic>/model/$(arg robot_namespace)/scan</topic>
+                <topic>$(arg robot_namespace)/scan</topic>
                 <update_rate>${two_d_lidar_update_rate}</update_rate>
                 <!-- Frame con namespace -->
@@ -86,10 +86,10 @@
                 <update_rate>30.0</update_rate>
                 <!-- Topic con namespace -->
-                <topic>/model/$(arg robot_namespace)/kinect_camera</topic>
+                <topic>$(arg robot_namespace)/kinect_camera</topic>
                 <!-- Frame con namespace -->
                 <gz_frame_id>$(arg robot_namespace)/kinect_camera</gz_frame_id>
                 <camera>
                     <!-- Camera info topic con namespace -->
-                    <camera_info_topic>/model/$(arg robot_namespace)/kinect_camera/camera_info</camera_info_topic>
+                    <camera_info_topic>$(arg robot_namespace)/kinect_camera/camera_info</camera_info_topic>
                     <horizontal_fov>${radians(camera_horizontal_fov)}</horizontal_fov>
                     <image>
@@ -115,5 +115,5 @@
             <visualize>true</visualize>
             <!-- Topic con namespace -->
-            <topic>/model/$(arg robot_namespace)/imu</topic>
+            <topic>$(arg robot_namespace)/imu</topic>
         </sensor>
     </gazebo>
@@ -128,6 +128,6 @@
                 <pose>0 -0.12 0 0 0 0</pose>
                 <!-- Topics con namespace -->
-                <topic>/model/$(arg robot_namespace)/stereo_camera/right/image_raw</topic>
-                <camera_info_topic>/model/$(arg robot_namespace)/stereo_camera/right/camera_info</camera_info_topic>
+                <topic>$(arg robot_namespace)/stereo_camera/right/image_raw</topic>
+                <camera_info_topic>$(arg robot_namespace)/stereo_camera/right/camera_info</camera_info_topic>
                 <horizontal_fov>1.3962634</horizontal_fov>
                 <image>
@@ -143,6 +143,6 @@
             <sensor type="camera" name="left">
                 <!-- Topics con namespace -->
-                <topic>/model/$(arg robot_namespace)/stereo_camera/left/image_raw</topic>
-                <camera_info_topic>/model/$(arg robot_namespace)/stereo_camera/left/camera_info</camera_info_topic>
+                <topic>$(arg robot_namespace)/stereo_camera/left/image_raw</topic>
+                <camera_info_topic>$(arg robot_namespace)/stereo_camera/left/camera_info</camera_info_topic>
                 <update_rate>10.0</update_rate>
                 <always_on>true</always_on>
