Commit message: add prefix  to robot

File: urdf/bcr_bot_ns.xacro (robot description, xacro)
@@ -41,25 +41,19 @@
     <xacro:arg name="odometry_source" default="world" />
     <xacro:property name="odometry_source" value="$(arg odometry_source)"/>
+    <xacro:property name="robot_namespace" value="$(arg robot_namespace)"/>
+    <xacro:property name="prefix" value="${robot_namespace + '/' if robot_namespace else ''}"/>
     <!-- ............................... LOAD MACROS ................................. -->
     <xacro:include filename="$(find bcr_bot)/urdf/materials.xacro"/>
     <xacro:include filename="$(find bcr_bot)/urdf/macros.xacro"/>
-    <xacro:if value="$(arg sim_gazebo)">
-        <xacro:include filename="$(find bcr_bot)/urdf/gazebo.xacro"/>
-    </xacro:if>
-    <xacro:if value="$(arg sim_ign)">
-        <xacro:include filename="$(find bcr_bot)/urdf/ign.xacro"/>
-    </xacro:if>
-    <xacro:if value="$(arg sim_gz)">
-        <xacro:include filename="$(find bcr_bot)/urdf/gz_ns.xacro"/>
-    </xacro:if>
+    <xacro:include filename="$(find bcr_bot)/urdf/gz_ns.xacro"/>
     <!-- ................................ BASE LINK .................................. -->
-    <link name="base_footprint"/>
-    <link name="base_link"/>
-    <joint name="base_joint" type="fixed">
-        <parent link="base_footprint"/>
-        <child link="base_link"/>
+    <link name="${prefix}base_footprint"/>
+    <link name="${prefix}base_link"/>
+    <joint name="${prefix}base_joint" type="fixed">
+        <parent link="${prefix}base_footprint"/>
+        <child link="${prefix}base_link"/>
         <origin xyz="0.0 0 ${chassis_height/2 + traction_wheel_radius}" rpy="0 0 0.0" />
     </joint>
-    <link name="chassis_link">
+    <link name="${prefix}chassis_link">
         <collision>
             <origin xyz="0 0 -0.05" rpy="0 0 0" />
@@ -79,19 +73,19 @@
         </inertial>
     </link>
-    <joint name="chassis_joint" type="fixed">
-        <parent link="base_link"/>
-        <child link="chassis_link"/>
+    <joint name="${prefix}chassis_joint" type="fixed">
+        <parent link="${prefix}base_link"/>
+        <child link="${prefix}chassis_link"/>
         <origin xyz="0.0 0 0" rpy="0 0 0.0" />
     </joint>
     <!-- ................................ WHEELS ..................................... -->
-    <xacro:trolley_wheel cardinality="front" dexterity="left" origin_x="${chassis_length/2}" origin_y="${trolley_track_width/2}" origin_z="-${trolley_wheel_radius+chassis_height/2}"/>
-    <xacro:trolley_wheel cardinality="front" dexterity="right" origin_x="${chassis_length/2}" origin_y="-${trolley_track_width/2}" origin_z="-${trolley_wheel_radius+chassis_height/2}"/>
-    <xacro:trolley_wheel cardinality="back" dexterity="left" origin_x="-${chassis_length/2}" origin_y="${trolley_track_width/2}" origin_z="-${trolley_wheel_radius+chassis_height/2}"/>
-    <xacro:trolley_wheel cardinality="back" dexterity="right" origin_x="-${chassis_length/2}" origin_y="-${trolley_track_width/2}" origin_z="-${trolley_wheel_radius+chassis_height/2}"/>
-    <xacro:traction_wheel cardinality="middle" dexterity="left" origin_x="0" origin_y="${traction_track_width/2}" origin_z="-${chassis_height/2+2*trolley_wheel_radius+eps-traction_wheel_radius}"/>
-    <xacro:traction_wheel cardinality="middle" dexterity="right" origin_x="0" origin_y="-${traction_track_width/2}" origin_z="-${chassis_height/2+2*trolley_wheel_radius+eps-traction_wheel_radius}"/>
+    <xacro:trolley_wheel cardinality="front" dexterity="left" origin_x="${chassis_length/2}" origin_y="${trolley_track_width/2}" origin_z="-${trolley_wheel_radius+chassis_height/2}" prefix="${prefix}"/>
+    <xacro:trolley_wheel cardinality="front" dexterity="right" origin_x="${chassis_length/2}" origin_y="-${trolley_track_width/2}" origin_z="-${trolley_wheel_radius+chassis_height/2}" prefix="${prefix}"/>
+    <xacro:trolley_wheel cardinality="back" dexterity="left" origin_x="-${chassis_length/2}" origin_y="${trolley_track_width/2}" origin_z="-${trolley_wheel_radius+chassis_height/2}" prefix="${prefix}"/>
+    <xacro:trolley_wheel cardinality="back" dexterity="right" origin_x="-${chassis_length/2}" origin_y="-${trolley_track_width/2}" origin_z="-${trolley_wheel_radius+chassis_height/2}" prefix="${prefix}"/>
+    <xacro:traction_wheel cardinality="middle" dexterity="left" origin_x="0" origin_y="${traction_track_width/2}" origin_z="-${chassis_height/2+2*trolley_wheel_radius+eps-traction_wheel_radius}" prefix="${prefix}"/>
+    <xacro:traction_wheel cardinality="middle" dexterity="right" origin_x="0" origin_y="-${traction_track_width/2}" origin_z="-${chassis_height/2+2*trolley_wheel_radius+eps-traction_wheel_radius}" prefix="${prefix}"/>
     <!-- ............................. 2D LIDAR ........................................ -->
     <xacro:if value="$(arg two_d_lidar_enabled)">
-        <link name="two_d_lidar">
+        <link name="${prefix}two_d_lidar">
             <collision>
                 <origin xyz="0 0 0" rpy="0 0 0" />
@@ -113,18 +107,18 @@
             </inertial>
         </link>
-        <joint name="two_d_lidar_joint" type="fixed">
-            <parent link="base_link"/>
-            <child link="two_d_lidar"/>
+        <joint name="${prefix}two_d_lidar_joint" type="fixed">
+            <parent link="${prefix}base_link"/>
+            <child link="${prefix}two_d_lidar"/>
             <origin xyz="0.0 0 0.08" rpy="0 0 0" />
         </joint>
-        <gazebo reference="two_d_lidar">
+        <gazebo reference="${prefix}two_d_lidar">
             <material>Gazebo/White</material>
         </gazebo>
     </xacro:if>
     <!-- ............................. IMU ........................................ -->
-    <link name="imu_frame"/>
-    <joint name="imu_joint" type="fixed">
-        <parent link="base_link"/>
-        <child link="imu_frame"/>
+    <link name="${prefix}imu_frame"/>
+    <joint name="${prefix}imu_joint" type="fixed">
+        <parent link="${prefix}base_link"/>
+        <child link="${prefix}imu_frame"/>
         <origin xyz="0.0 0.0 0.08" rpy="0.0 0.0 0.0"/>
     </joint>
@@ -132,5 +126,5 @@
     <xacro:if value="$(arg camera_enabled)">
         <!-- KINECT CAMERA -->
-        <link name="kinect_camera">
+        <link name="${prefix}kinect_camera">
             <collision>
                 <origin xyz="0 0 0" rpy="0 0 0" />
@@ -151,14 +145,14 @@
             </inertial>
         </link>
-        <joint name="kinect_camera_joint" type="fixed">
+        <joint name="${prefix}kinect_camera_joint" type="fixed">
             <origin rpy="0 0 0" xyz="${chassis_length/2} 0 ${chassis_height/7}"/>
-            <parent link="base_link"/>
-            <child link="kinect_camera"/>
-        </joint>
-        <link name="kinect_camera_optical"/>
-        <joint name="kinect_camera_optical_joint" type="fixed">
+            <parent link="${prefix}base_link"/>
+            <child link="${prefix}kinect_camera"/>
+        </joint>
+        <link name="${prefix}kinect_camera_optical"/>
+        <joint name="${prefix}kinect_camera_optical_joint" type="fixed">
             <origin xyz="0 0 0" rpy="${-pi/2} 0 ${-pi/2}"/>
-            <parent link="kinect_camera"/>
-            <child link="kinect_camera_optical"/>
+            <parent link="${prefix}kinect_camera"/>
+            <child link="${prefix}kinect_camera_optical"/>
         </joint>
     </xacro:if>
@@ -166,5 +160,5 @@
     <xacro:if value="$(arg stereo_camera_enabled)">
         <!-- STEREO CAMERA -->
-        <link name="stereo_camera">
+        <link name="${prefix}stereo_camera">
             <collision>
                 <origin xyz="0 0 0" rpy="0 0 0" />
@@ -185,18 +179,18 @@
             </inertial>
         </link>
-        <joint name="stereo_camera_joint" type="fixed">
+        <joint name="${prefix}stereo_camera_joint" type="fixed">
             <origin rpy="0 0 0" xyz="${chassis_length/2} 0 ${chassis_height/7}"/>
-            <parent link="base_link"/>
-            <child link="stereo_camera"/>
-        </joint>
-        <link name="stereo_camera_optical"/>
-        <joint name="stereo_camera_optical_joint" type="fixed">
+            <parent link="${prefix}base_link"/>
+            <child link="${prefix}stereo_camera"/>
+        </joint>
+        <link name="${prefix}stereo_camera_optical"/>
+        <joint name="${prefix}stereo_camera_optical_joint" type="fixed">
             <origin xyz="0 0 0" rpy="${-pi/2} 0 ${-pi/2}"/>
-            <parent link="stereo_camera"/>
-            <child link="stereo_camera_optical"/>
+            <parent link="${prefix}stereo_camera"/>
+            <child link="${prefix}stereo_camera_optical"/>
         </joint>
     </xacro:if>
     <!-- ............................. ROOF ........................................ -->
-    <link name="roof_link">
+    <link name="${prefix}roof_link">
         <collision>
             <origin xyz="0 0 0" rpy="0 0 0" />
@@ -210,12 +204,12 @@
         </inertial>
     </link>
-    <joint name="roof_joint" type="fixed">
-        <parent link="chassis_link"/>
-        <child link="roof_link"/>
+    <joint name="${prefix}roof_joint" type="fixed">
+        <parent link="${prefix}chassis_link"/>
+        <child link="${prefix}roof_link"/>
         <origin xyz="0 0 0.16" rpy="0 0 0" />
     </joint>
     <!-- ............................. CONVEYOR ........................................ -->
     <xacro:if value="$(arg conveyor_enabled)">
-        <link name="conveyor_belt">
+        <link name="${prefix}conveyor_belt">
             <collision>
                 <origin xyz="0 0 0" rpy="0 0 0" />
@@ -235,7 +229,7 @@
             </inertial>
         </link>
-        <joint name="conveyor_joint" type="fixed">
-            <parent link="base_link"/>
-            <child link="conveyor_belt"/>
+        <joint name="${prefix}conveyor_joint" type="fixed">
+            <parent link="${prefix}base_link"/>
+            <child link="${prefix}conveyor_belt"/>
             <origin xyz="0 0 0.25" rpy="0 0 0" />
         </joint>

File: urdf/gz_ns.xacro (robot description, xacro)
@@ -3,4 +3,6 @@
     <!-- Argumento para el namespace del robot -->
     <xacro:arg name="robot_namespace" default="bcr_bot"/>
+    <xacro:property name="robot_namespace" value="$(arg robot_namespace)"/>
+    <xacro:property name="prefix" value="${robot_namespace + '/' if robot_namespace else ''}"/>
     <!-- ........................... SENSOR PLUGIN ................................... -->
     <gazebo>
@@ -14,6 +16,6 @@
         <!-- ........................... DIFFERENTIAL DRIVE PLUGIN ................................... -->
         <plugin filename="gz-sim-diff-drive-system" name="gz::sim::systems::DiffDrive">
-            <left_joint>middle_left_wheel_joint</left_joint>
-            <right_joint>middle_right_wheel_joint</right_joint>
+            <left_joint>${prefix}middle_left_wheel_joint</left_joint>
+            <right_joint>${prefix}middle_right_wheel_joint</right_joint>
             <wheel_separation>${traction_track_width+traction_wheel_width-0.01}</wheel_separation>
             <wheel_radius>${traction_wheel_radius+0.01}</wheel_radius>
@@ -48,11 +50,10 @@
     <!-- ........................... 2D LIDAR config ................................... -->
     <xacro:if value="$(arg two_d_lidar_enabled)">
-        <gazebo reference="two_d_lidar">
+        <gazebo reference="${prefix}two_d_lidar">
             <sensor name='gpu_lidar' type='gpu_lidar'>
-                <!-- Topic con namespace -->
+                <pose>0 0 0 0 0 0</pose>
+                <!-- <pose relative_to="${prefix}two_d_lidar">0 0 0 0 0 0</pose> -->
                 <topic>$(arg robot_namespace)/scan</topic>
                 <update_rate>${two_d_lidar_update_rate}</update_rate>
-                <!-- Frame con namespace -->
-                <gz_frame_id>$(arg robot_namespace)/two_d_lidar</gz_frame_id>
                 <lidar>
                     <scan>
@@ -82,14 +83,14 @@
     <!-- ........................... CAMERA config ................................... -->
     <xacro:if value="$(arg camera_enabled)">
-        <gazebo reference="kinect_camera">
+        <gazebo reference="${prefix}kinect_camera">
             <sensor type="depth_camera" name="kinect_camera">
                 <update_rate>30.0</update_rate>
+                <always_on>1</always_on>
+                <visualize>true</visualize>
                 <!-- Topic con namespace -->
                 <topic>$(arg robot_namespace)/kinect_camera</topic>
-                <!-- Frame con namespace -->
-                <gz_frame_id>$(arg robot_namespace)/kinect_camera</gz_frame_id>
-                <camera>
-                    <!-- Camera info topic con namespace -->
-                    <camera_info_topic>$(arg robot_namespace)/kinect_camera/camera_info</camera_info_topic>
+                <!-- Pose del sensor relativo al link -->
+                <pose>0 0 0 0 0 0</pose>
+                <camera name="kinect_camera">
                     <horizontal_fov>${radians(camera_horizontal_fov)}</horizontal_fov>
                     <image>
@@ -102,4 +103,27 @@
                         <far>8.0</far>
                     </clip>
+                    <depth_camera>
+                        <clip>
+                            <near>0.05</near>
+                            <far>8.0</far>
+                        </clip>
+                    </depth_camera>
+                    <distortion>
+                        <k1>0.0</k1>
+                        <k2>0.0</k2>
+                        <k3>0.0</k3>
+                        <p1>0.0</p1>
+                        <p2>0.0</p2>
+                        <center>0.5 0.5</center>
+                    </distortion>
+                    <lens>
+                        <intrinsics>
+                            <fx>554.25</fx>
+                            <fy>554.25</fy>
+                            <cx>320.5</cx>
+                            <cy>240.5</cy>
+                            <s>0</s>
+                        </intrinsics>
+                    </lens>
                 </camera>
             </sensor>
@@ -107,10 +131,8 @@
     </xacro:if>
     <!-- ........................... IMU config ................................... -->
-    <gazebo reference="imu_frame">
+    <gazebo reference="${prefix}imu_frame">
         <sensor name="imu_sensor" type="imu">
             <always_on>1</always_on>
             <update_rate>1</update_rate>
-            <!-- Frame con namespace -->
-            <gz_frame_id>$(arg robot_namespace)/imu_frame</gz_frame_id>
             <visualize>true</visualize>
             <!-- Topic con namespace -->
@@ -120,44 +142,42 @@
     <!-- ........................... Stereo camera ................................... -->
     <xacro:if value="$(arg stereo_camera_enabled)">
-        <gazebo reference="stereo_camera">
+        <gazebo reference="${prefix}stereo_camera">
             <sensor type="camera" name="right">
                 <update_rate>10.0</update_rate>
                 <always_on>true</always_on>
-                <!-- Frame con namespace -->
-                <gz_frame_id>$(arg robot_namespace)/stereo_camera_optical</gz_frame_id>
                 <pose>0 -0.12 0 0 0 0</pose>
                 <!-- Topics con namespace -->
                 <topic>$(arg robot_namespace)/stereo_camera/right/image_raw</topic>
-                <camera_info_topic>$(arg robot_namespace)/stereo_camera/right/camera_info</camera_info_topic>
-                <horizontal_fov>1.3962634</horizontal_fov>
-                <image>
-                    <width>1024</width>
-                    <height>1024</height>
-                    <format>R8G8B8</format>
-                </image>
-                <clip>
-                    <near>0.3</near>
-                    <far>20</far>
-                </clip>
+                <camera name="right_camera">
+                    <horizontal_fov>1.3962634</horizontal_fov>
+                    <image>
+                        <width>1024</width>
+                        <height>1024</height>
+                        <format>R8G8B8</format>
+                    </image>
+                    <clip>
+                        <near>0.3</near>
+                        <far>20</far>
+                    </clip>
+                </camera>
             </sensor>
             <sensor type="camera" name="left">
                 <!-- Topics con namespace -->
                 <topic>$(arg robot_namespace)/stereo_camera/left/image_raw</topic>
-                <camera_info_topic>$(arg robot_namespace)/stereo_camera/left/camera_info</camera_info_topic>
                 <update_rate>10.0</update_rate>
                 <always_on>true</always_on>
-                <!-- Frame con namespace -->
-                <gz_frame_id>$(arg robot_namespace)/stereo_camera_optical</gz_frame_id>
                 <pose>0 0 0 0 0 0</pose>
-                <horizontal_fov>1.3962634</horizontal_fov>
-                <image>
-                    <width>1024</width>
-                    <height>1024</height>
-                    <format>R8G8B8</format>
-                </image>
-                <clip>
-                    <near>0.3</near>
-                    <far>20</far>
-                </clip>
+                <camera name="left_camera">
+                    <horizontal_fov>1.3962634</horizontal_fov>
+                    <image>
+                        <width>1024</width>
+                        <height>1024</height>
+                        <format>R8G8B8</format>
+                    </image>
+                    <clip>
+                        <near>0.3</near>
+                        <far>20</far>
+                    </clip>
+                </camera>
             </sensor>
         </gazebo>

File: urdf/macros.xacro (robot description, xacro)
@@ -12,6 +12,6 @@
     </xacro:macro>
     <!-- ............................... TROLLEY WHEEL DEFINITION .............................. -->
-    <xacro:macro name="trolley_wheel" params="cardinality dexterity origin_x origin_y origin_z">
-        <link name="${cardinality}_${dexterity}_wheel">
+    <xacro:macro name="trolley_wheel" params="cardinality dexterity origin_x origin_y origin_z prefix:=''">
+        <link name="${prefix}${cardinality}_${dexterity}_wheel">
             <collision>
                 <origin xyz="0 0 0" rpy="0 ${pi/2} ${pi/2}" />
@@ -27,16 +27,16 @@
             <mu>0.0</mu>
         </link>
-        <joint name="${cardinality}_${dexterity}_wheel_joint" type="fixed">
-            <parent link="base_link"/>
-            <child link="${cardinality}_${dexterity}_wheel"/>
+        <joint name="${prefix}${cardinality}_${dexterity}_wheel_joint" type="fixed">
+            <parent link="${prefix}base_link"/>
+            <child link="${prefix}${cardinality}_${dexterity}_wheel"/>
             <origin xyz="${origin_x} ${origin_y} ${origin_z}" rpy="0 0 0" />
             <axis xyz="0 1 0" rpy="0 0 0" />
         </joint>
-        <gazebo reference="${cardinality}_${dexterity}_wheel">
+        <gazebo reference="${prefix}${cardinality}_${dexterity}_wheel">
             <material>Gazebo/Black</material>
         </gazebo>
     </xacro:macro>
-    <xacro:macro name="traction_wheel" params="cardinality dexterity origin_x origin_y origin_z">
-        <link name="${cardinality}_${dexterity}_wheel">
+    <xacro:macro name="traction_wheel" params="cardinality dexterity origin_x origin_y origin_z prefix:=''">
+        <link name="${prefix}${cardinality}_${dexterity}_wheel">
             <collision>
                 <origin xyz="0 0 0" rpy="0 ${pi/2} ${pi/2}" />
@@ -53,11 +53,11 @@
             <mu>5.0</mu>
         </link>
-        <joint name="${cardinality}_${dexterity}_wheel_joint" type="continuous">
-            <parent link="base_link"/>
-            <child link="${cardinality}_${dexterity}_wheel"/>
+        <joint name="${prefix}${cardinality}_${dexterity}_wheel_joint" type="continuous">
+            <parent link="${prefix}base_link"/>
+            <child link="${prefix}${cardinality}_${dexterity}_wheel"/>
             <origin xyz="${origin_x} ${origin_y} ${origin_z}" rpy="0 0 0" />
             <axis xyz="0 1 0" rpy="0 0 0" />
         </joint>
-        <gazebo reference="${cardinality}_${dexterity}_wheel">
+        <gazebo reference="${prefix}${cardinality}_${dexterity}_wheel">
             <material>Gazebo/Black</material>
         </gazebo>
